File: Hardware/CV-Module CAD/CV-module-schematics.sch (EAGLE design)
At the start: 12 parts, among them U1 AD5611BKSZ, U2 AD5611BKSZ, U3 AD5611BKSZ, U4 AD5611BKSZ, U5 AD5611BKSZ, U6 AD5611BKSZ, U7 AD5611BKSZ, U8 AD5611BKSZ

Commit message: working on eagle-project
Parts:
- added C1, C2, C3, C4, C5, C6, C7, C8: 10uF, resistor:C-EUC1206
- added C10, C11, C12, C13, C14, C15, C16, C9: 0,1uF, resistor:C-EUC0603
- added U$1: CD4051BM96, halo-electronics:CD4051BM96
- added U$2: POWER_SIMPLE10, eurorack:POWER_SIMPLE10
Connections:
- new net SYNC1: U$1.OUT0, U1.!SYNC
- new net SYNC2: U$1.OUT1, U2.!SYNC
- new net SYNC3: U$1.OUT2, U3.!SYNC
- new net SYNC4: U$1.OUT3, U4.!SYNC
- new net SYNC5: U$1.OUT4, U5.!SYNC
- new net SYNC6: U$1.OUT5, U6.!SYNC
- new net SYNC7: U$1.OUT6, U7.!SYNC
- new net SYNC8: U$1.OUT7, U8.!SYNC
- new net VDAC1: U1.VOUT
- new net VDAC2: U2.VOUT
- new net VDAC3: U3.VOUT
- new net VDAC4: U4.VOUT
- new net VDAC5: U5.VOUT
- new net VDAC6: U6.VOUT
- new net VDAC7: U7.VOUT
- new net VDAC8: U8.VOUT
- net GND: now also C1.2, C10.2, C11.2, C12.2, C13.2, C14.2, C15.2, C16.2, C2.2, C3.2, C4.2, C5.2, C6.2, C7.2, C8.2, C9.2
- net VDD: now also C1.1, C10.1, C11.1, C12.1, C13.1, C15.1, C16.1, C2.1, C3.1, C4.1, C5.1, C6.1, C7.1, C8.1, C9.1, IC1.OUT, U1.VDD, U2.VDD, U4.VDD, U5.VDD, U6.VDD, U7.VDD, U8.VDD
Other:
- moved on the sheet: IC1, U5, U6, U7, U8

Commit message: HW-design phase
Parts:
- removed U$2: POWER_SIMPLE10, eurorack:POWER_SIMPLE10
- added C17: 10uF, resistor:C-EUC1206
- added R10, R11, R4, R5, R6, R7, R8, R9: 20k, resistor:R-US_M1206
- added U$3: POWER, eurorack:POWER
Connections:
- new net N$3: C17.1, IC1.EN, IC1.IN, U$3.+12V
- new net VCC: C1.1, C10.1, C11.1, C12.1, C13.1, C15.1, C16.1, C2.1, C3.1, C4.1, C5.1, C6.1, C7.1, C8.1, C9.1, IC1.OUT, U1.VDD, U2.VDD, U3.VDD, U4.VDD, U5.VDD, U6.VDD, U7.VDD, U8.VDD
- net GND: now also C17.2, IC1.GND, R11.2, R4.2, R5.2, R6.2, R7.2, R8.2, R9.2, U$1.INH, U$1.VEE, U$1.VSS, U$3.GND
- net SYNC1: now also R4.1
- net SYNC2: now also R5.1
- net SYNC3: now also R6.1
- net SYNC4: now also R7.1
- net SYNC5: now also R8.1
- net SYNC6: now also R9.1
- net SYNC7: now also R10.1
- net SYNC8: now also R11.1
- net VDD: now also U$1.IN, U$1.VDD; no longer C1.1, C10.1, C11.1, C12.1, C13.1, C15.1, C16.1, C2.1, C3.1, C4.1, C5.1, C6.1, C7.1, C8.1, C9.1, IC1.OUT, U1.VDD, U2.VDD, U3.VDD, U4.VDD, U5.VDD, U6.VDD, U7.VDD, U8.VDD
Other:
- note added: "- Analog out signal conditioning (op-amps)"
- note added: "MULTIPLEXER"
- note added: "Todo:"
- note added: "output to raspberry pi (usb-micro usb tms)"

Commit message: eagle project forward
Parts:
- added IC2, IC3, IC4, IC5: LM358D, linear:LM358D
- added JP1: (no value), pinhead:PINHD-2X4
- added R12, R13, R14, R15, R16, R17, R18, R19, R20, R21, R22, R23, R24, R25, R26, R27: 10k, resistor:R-US_R0603
- added R28, R29, R30, R31, R32, R33, R34, R35: (no value), pot:TRIM_EU-3223W
- added U9: (no value), SparkFun-PowerIC:V_REG_LM1117SOT223
Connections:
- new net +5V: R28.S, U9.OUT, U9.OUT@1
- new net N$5: R12.1, R28.A
- net GND: now also U9.ADJ
- net N$3: now also U9.IN

Commit message: HW schematics and layout +parts updated
Parts:
- removed R10, R11, R9: 20k, resistor:R-US_M1206
- added C18, C19: 10uF, resistor:C-EUC1206
- added JP2: (no value), pinhead:PINHD-2X3
- added R36, R37, R38, R39, R40, R41, R42, R43: 1k, resistor:R-US_R0603
- R1, R2, R3: value (none) -> 20k; device resistor:R-US_R1206 -> rcl:R-US_R0603
- R12, R14, R16, R18, R20, R22, R24, R26: value 10k -> 9.53k
- R4, R5, R6, R7, R8: device resistor:R-US_M1206 -> rcl:R-US_R0603
Connections:
- removed net N$3: C17.1, IC1.EN, IC1.IN, U$3.+12V, U9.IN
- new net +12VDC: C17.1, C19.1, IC1.EN, IC1.IN, IC2P.V+, IC3P.V+, IC4P.V+, IC5P.V+, U$3.+12V, U9.IN
- new net -12VDC: IC2P.V-, IC3P.V-, IC4P.V-, IC5P.V-, U$3.-12V
- new net CTRL1: U$1.A
- new net CTRL2: U$1.B
- new net CTRL3: U$1.C
- new net CV1: R36.2
- new net CV2: R37.2
- new net CV3: R38.2
- new net CV4: R39.2
- new net CV5: JP1.2, R40.2
- new net CV6: JP1.4, R41.2
- new net CV7: JP1.6, R42.2
- new net CV8: JP1.8, R43.2
- new net N$10: R16.1, R30.A
- new net N$11: IC3B.-IN, R18.2, R19.1
- new net N$12: R18.1, R31.A
- new net N$13: IC3B.OUT, R19.2, R39.1
- new net N$14: IC3A.OUT, R17.2, R38.1
- new net N$15: IC2B.OUT, R15.2, R37.1
- new net N$16: IC4A.-IN, R20.2, R21.1
- new net N$17: IC4A.OUT, R21.2, R40.1
- new net N$18: IC4B.OUT, R23.2, R41.1
- new net N$19: IC4B.-IN, R22.2, R23.1
- new net N$20: IC5A.-IN, R24.2, R25.1
- new net N$21: IC5A.OUT, R25.2, R42.1
- new net N$22: R24.1, R34.A
- new net N$23: IC5B.-IN, R26.2, R27.1
- new net N$24: IC5B.OUT, R27.2, R43.1
- new net N$25: R26.1, R35.A
- new net N$26: R20.1, R32.A
- new net N$27: R22.1, R33.A
- new net N$4: IC2A.-IN, R12.2, R13.1
- new net N$6: IC2A.OUT, R13.2, R36.1
- new net N$7: R14.1, R29.A
- new net N$8: IC2B.-IN, R14.2, R15.1
- new net N$9: IC3A.-IN, R16.2, R17.1
- net +5V: now also C18.1, R29.S, R30.S, R31.S, R32.S, R33.S, R34.S, R35.S
- net GND: now also C18.2, C19.2, R1.2, R2.2, R3.2; no longer R11.2, R9.2
- net N$1: now also JP2.2, U1.SDIN, U2.SDIN, U3.SDIN, U5.SDIN, U6.SDIN, U7.SDIN, U8.SDIN; no longer R2.2
- net N$2: now also JP2.4, U1.SCLK, U2.SCLK, U3.SCLK, U5.SCLK, U6.SCLK, U7.SCLK, U8.SCLK; no longer R1.1
- net SYNC1: now also R1.1; no longer R4.1
- net SYNC2: now also R2.1; no longer R5.1
- net SYNC3: now also R3.1; no longer R6.1
- net SYNC4: now also R4.1; no longer R7.1
- net SYNC5: now also R5.1; no longer R8.1
- net SYNC6: now also R6.1; no longer R9.1
- net SYNC7: now also R7.1; no longer R10.1
- net SYNC8: now also R8.1; no longer R11.1
- net VDAC1: now also IC2A.+IN
- net VDAC2: now also IC2B.+IN
- net VDAC3: now also IC3A.+IN
- net VDAC4: now also IC3B.+IN
- net VDAC5: now also IC4A.+IN
- net VDAC6: now also IC4B.+IN
- net VDAC7: now also IC5A.+IN
- net VDAC8: now also IC5B.+IN
Other:
- note added: "DAC:s"
- note added: "To Raspberry Pi"
- note added: "Voltage reference for DAC"
- note added: "Voltage regulator for OP-amps"
- note removed: "- Analog out signal conditioning (op-amps)"
- note removed: "Todo:"
- note removed: "output to raspberry pi (usb-micro usb tms)"
- moved on the sheet: IC2B, IC3A, IC3B, IC4A, IC4B, IC5A, IC5B, R1, R16, R17, R18, R19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

Commit message: Schema and Layout
Parts:
- added C20, C21: 0.1uF, rcl:C-EUC0603
- added C22, C23: 10uF, rcl:CPOLRAD
- added C24, C25: 1uF, rcl:CPOLRAD
- added U$2: PCM1808PW, Pekkas_libraries:PCM1808PW
Changed lines of the file:
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@@
 <layer number="102" name="Vscore" color="7" fill="1" visible="no" active="yes"/>
 <layer number="103" name="tMap" color="7" fill="1" visible="no" active="yes"/>
-<layer number="104" name="Name" color="16" fill="1" visible="no" active="yes"/>
+<layer number="104" name="Name" color="16" fill="1" visible="yes" active="yes"/>
 <layer number="105" name="tPlate" color="7" fill="1" visible="no" active="yes"/>
 <layer number="106" name="bPlate" color="7" fill="1" visible="no" active="yes"/>
@@
 <part name="R7" library="rcl" deviceset="R-US_" device="R0603" value="20k"/>
 <part name="R8" library="rcl" deviceset="R-US_" device="R0603" value="20k"/>
+<part name="U$2" library="Pekkas_libraries" deviceset="PCM1808PW" device=""/>
+<part name="C20" library="rcl" deviceset="C-EU" device="C0603" value="0.1uF"/>
+<part name="C21" library="rcl" deviceset="C-EU" device="C0603" value="0.1uF"/>
+<part name="C22" library="rcl" deviceset="CPOLRAD" device="" value="10uF"/>
+<part name="C23" library="rcl" deviceset="CPOLRAD" device="" value="10uF"/>
+<part name="C24" library="rcl" deviceset="CPOLRAD" device="" value="1uF"/>
+<part name="C25" library="rcl" deviceset="CPOLRAD" device="" value="1uF"/>
 </parts>
 <sheets>
@@
 </nets>
 </sheet>
+<sheet>
+<plain>
+</plain>
+<instances>
+<instance part="U$2" gate="G$1" x="71.12" y="53.34"/>
+<instance part="C20" gate="G$1" x="10.16" y="71.12"/>
+<instance part="C21" gate="G$1" x="10.16" y="58.42"/>
+<instance part="C22" gate="G$1" x="33.02" y="71.12"/>
+<instance part="C23" gate="G$1" x="27.94" y="50.8"/>
+<instance part="C24" gate="G$1" x="35.56" y="30.48"/>
+<instance part="C25" gate="G$1" x="55.88" y="17.78"/>
+</instances>
+<busses>
+</busses>
+<nets>
+</nets>
+</sheet>

Commit message: layout forward
Parts:
- removed U$2: PCM1808PW, Pekkas_libraries:PCM1808PW
- added C26, C27, C30: 0.1uF, rcl:C-EUC0603
- added C28: (no value), rcl:C-USC1206
- added C29: 10uF, rcl:CPOLRAD
- added IC6: (no value), SparkFun-PowerIC:V_REG_TPS76433SOT23-5
- added JP3: (no value), pinhead:PINHD-2X3
- added PCM1808: PCM1808PW, Pekkas_libraries:PCM1808PW
- added TLV71333: TVL713, Pekkas_libraries:TVL713
Connections:
- new net 3V3: C21.1, C23.+, C26.1, PCM1808.VDD, TLV71333.OUT
- new net 5VCC: C20.1, C22.+, IC6.OUT, PCM1808.VCC
- new net 5VCON: C27.1, TLV71333.EN, TLV71333.IN, U$3.+5V
- new net AGND: C20.2, C22.-
- new net N$28: C25.+, PCM1808.VINL
- new net N$3: C24.+, PCM1808.VINR
- new net N$31: C29.+, C30.1
- net +12VDC: now also C28.1, IC6.EN, IC6.IN
- net GND: now also C21.2, C23.-, C26.2, C27.2, C28.2, C29.-, C30.2, IC6.GND, PCM1808.AGND, PCM1808.DGND, PCM1808.FMT, PCM1808.MD0, PCM1808.MD1, TLV71333.GND
Other:
- note added: "Analog to digital conversion"
- note added: "CV outputs"
- note added: "Caps for pcm1808"
- note added: "Control-Voltage signal conditioning"
- note added: "Digital to analog conversion"
- note added: "PCM1808"
- moved on the sheet: C20, C21, C22, C23, C24, C25

Commit message: Schema and layout design
Parts:
- added C31, C32: 10uF, resistor:C-EUC1206
- added CDCS502PW: CDCS502, components:CDCS502
- added Q1: (no value), Pekkas_libraries:XTAL
- added U$2: TVL713, Pekkas_libraries:TVL713
Connections:
- removed net VDD: U$1.IN, U$1.VDD
- new net 3V3MUX: C31.1, U$1.IN, U$1.VDD, U$2.OUT
- new net N$29: CDCS502PW.XIN, Q1.1
- new net N$30: CDCS502PW.XOUT, Q1.2
- new net N$32: CDCS502PW.CLK_OUT, PCM1808.SCK
- new net N$33: JP3.1, PCM1808.LRCK
- new net N$34: JP3.2, PCM1808.DOUT
- new net N$35: JP3.3, PCM1808.BCK
- net 3V3: now also CDCS502PW.VDD
- net 5VCON: now also C32.1, U$2.EN, U$2.IN
- net CTRL1: now also JP2.1
- net CTRL2: now also JP2.3
- net CTRL3: now also JP2.5
- net GND: now also C31.2, C32.2, CDCS502PW.FS, CDCS502PW.GND, CDCS502PW.SSC_SEL_0, CDCS502PW.SSC_SEL_1, JP3.4, U$2.GND
Other:
- note added: "Connector to RasPi"
- note added: "Voltage regulator for MULTIPLEXER"
- moved on the sheet: JP2, JP3

Commit message: layout&schematics
Connections:
- net N$1: now also U4.SDIN
- net N$2: now also U4.SCLK
- net SYNC6: now also U8.!SYNC; no longer U6.!SYNC
- net SYNC7: now also U6.!SYNC; no longer U7.!SYNC
- net SYNC8: now also U7.!SYNC; no longer U8.!SYNC
- net VCC: now also C14.1
Other:
- moved on the sheet: C14
Changed lines of the file:
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@@
 <instance part="C12" gate="G$1" x="-33.02" y="48.26"/>
 <instance part="C13" gate="G$1" x="-25.4" y="48.26"/>
-<instance part="C14" gate="G$1" x="-17.78" y="48.26"/>
+<instance part="C14" gate="G$1" x="-17.78" y="45.72"/>
 <instance part="C15" gate="G$1" x="-10.16" y="48.26"/>
 <instance part="C16" gate="G$1" x="-2.54" y="48.26"/>
@@
 <junction x="-10.16" y="38.1"/>
 <pinref part="C14" gate="G$1" pin="2"/>
-<wire x1="-17.78" y1="38.1" x2="-17.78" y2="43.18" width="0.1524" layer="91"/>
+<wire x1="-17.78" y1="38.1" x2="-17.78" y2="40.64" width="0.1524" layer="91"/>
 <junction x="-17.78" y="38.1"/>
 <pinref part="C13" gate="G$1" pin="2"/>
@@
 </segment>
 <segment>
+<pinref part="U8" gate="A" pin="!SYNC"/>
+<wire x1="104.14" y1="-10.16" x2="93.98" y2="-10.16" width="0.1524" layer="91"/>
+</segment>
+</net>
+<net name="SYNC7" class="0">
+<segment>
+<pinref part="U$1" gate="G$1" pin="OUT6"/>
+<wire x1="-5.08" y1="78.74" x2="2.54" y2="78.74" width="0.1524" layer="91"/>
+</segment>
+<segment>
+<wire x1="78.74" y1="111.76" x2="78.74" y2="109.22" width="0.1524" layer="91"/>
+<pinref part="R7" gate="G$1" pin="1"/>
+</segment>
+<segment>
 <pinref part="U6" gate="A" pin="!SYNC"/>
 <wire x1="104.14" y1="53.34" x2="93.98" y2="53.34" width="0.1524" layer="91"/>
 </segment>
 </net>
-<net name="SYNC7" class="0">
-<segment>
-<pinref part="U$1" gate="G$1" pin="OUT6"/>
-<wire x1="-5.08" y1="78.74" x2="2.54" y2="78.74" width="0.1524" layer="91"/>
-</segment>
-<segment>
-<wire x1="78.74" y1="111.76" x2="78.74" y2="109.22" width="0.1524" layer="91"/>
-<pinref part="R7" gate="G$1" pin="1"/>
+<net name="SYNC8" class="0">
+<segment>
+<pinref part="U$1" gate="G$1" pin="OUT7"/>
+<wire x1="-5.08" y1="76.2" x2="2.54" y2="76.2" width="0.1524" layer="91"/>
+</segment>
+<segment>
+<wire x1="86.36" y1="111.76" x2="86.36" y2="109.22" width="0.1524" layer="91"/>
+<pinref part="R8" gate="G$1" pin="1"/>
 </segment>
 <segment>
 <pinref part="U7" gate="A" pin="!SYNC"/>
 <wire x1="104.14" y1="22.86" x2="93.98" y2="22.86" width="0.1524" layer="91"/>
-</segment>
-</net>
-<net name="SYNC8" class="0">
-<segment>
-<pinref part="U$1" gate="G$1" pin="OUT7"/>
-<wire x1="-5.08" y1="76.2" x2="2.54" y2="76.2" width="0.1524" layer="91"/>
-</segment>
-<segment>
-<wire x1="86.36" y1="111.76" x2="86.36" y2="109.22" width="0.1524" layer="91"/>
-<pinref part="R8" gate="G$1" pin="1"/>
-</segment>
-<segment>
-<pinref part="U8" gate="A" pin="!SYNC"/>
-<wire x1="104.14" y1="-10.16" x2="93.98" y2="-10.16" width="0.1524" layer="91"/>
 </segment>
 </net>
@@
 <wire x1="-60.96" y1="58.42" x2="-60.96" y2="53.34" width="0.1524" layer="91"/>
 <junction x="-60.96" y="53.34"/>
+<pinref part="C14" gate="G$1" pin="1"/>
 </segment>
 <segment>
@@
 <wire x1="86.36" y1="-12.7" x2="86.36" y2="-48.26" width="0.1524" layer="91"/>
 <wire x1="86.36" y1="-48.26" x2="10.16" y2="-48.26" width="0.1524" layer="91"/>
-<wire x1="10.16" y1="-48.26" x2="10.16" y2="12.7" width="0.1524" layer="91"/>
+<wire x1="10.16" y1="-48.26" x2="10.16" y2="-12.7" width="0.1524" layer="91"/>
 <junction x="10.16" y="12.7"/>
 <pinref part="U6" gate="A" pin="SDIN"/>
+<wire x1="10.16" y1="-12.7" x2="10.16" y2="12.7" width="0.1524" layer="91"/>
 <wire x1="104.14" y1="50.8" x2="86.36" y2="50.8" width="0.1524" layer="91"/>
 <junction x="86.36" y="50.8"/>
@@
 <wire x1="104.14" y1="-12.7" x2="86.36" y2="-12.7" width="0.1524" layer="91"/>
 <junction x="86.36" y="-12.7"/>
+<pinref part="U4" gate="A" pin="SDIN"/>
+<wire x1="43.18" y1="-12.7" x2="10.16" y2="-12.7" width="0.1524" layer="91"/>
+<junction x="10.16" y="-12.7"/>
 </segment>
 </net>
@@
 <wire x1="88.9" y1="-15.24" x2="88.9" y2="-45.72" width="0.1524" layer="91"/>
 <wire x1="88.9" y1="-45.72" x2="17.78" y2="-45.72" width="0.1524" layer="91"/>
-<wire x1="17.78" y1="-45.72" x2="17.78" y2="10.16" width="0.1524" layer="91"/>
+<wire x1="17.78" y1="-45.72" x2="17.78" y2="-15.24" width="0.1524" layer="91"/>
 <junction x="17.78" y="10.16"/>
 <pinref part="U6" gate="A" pin="SCLK"/>
+<wire x1="17.78" y1="-15.24" x2="17.78" y2="10.16" width="0.1524" layer="91"/>
 <wire x1="104.14" y1="48.26" x2="88.9" y2="48.26" width="0.1524" layer="91"/>
 <junction x="88.9" y="48.26"/>
@@
 <wire x1="104.14" y1="-15.24" x2="88.9" y2="-15.24" width="0.1524" layer="91"/>
 <junction x="88.9" y="-15.24"/>
-</segment>
-</net>
+<pinref part="U4" gate="A" pin="SCLK"/>
+<wire x1="43.18" y1="-15.24" x2="17.78" y2="-15.24" width="0.1524" layer="91"/>
+<junction x="17.78" y="-15.24"/>
+</segment>
+</net>
