File: Hardware/CV-Module CAD/CV-module-schematics.sch (EAGLE design)
At the start: 97 parts, among them IC2 LM358D, IC3 LM358D, IC4 LM358D, IC5 LM358D, U1 AD5611BKSZ, U2 AD5611BKSZ, U3 AD5611BKSZ, U4 AD5611BKSZ, U5 AD5611BKSZ, U6 AD5611BKSZ, U7 AD5611BKSZ, U8 AD5611BKSZ

Commit message: HW
Connections:
- net CV1: now also JP1.1
- net CV2: now also JP1.3
- net CV3: now also JP1.5; no longer R38.2
- net CV4: now also JP1.7, R38.2
Changed lines of the file:
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@@
 <net name="CV1" class="0">
+<segment>
+<wire x1="78.74" y1="-30.48" x2="76.2" y2="-30.48" width="0.1524" layer="91"/>
+<pinref part="JP1" gate="A" pin="1"/>
+<wire x1="76.2" y1="-30.48" x2="63.5" y2="-30.48" width="0.1524" layer="91"/>
+<junction x="76.2" y="-30.48"/>
+</segment>
 <segment>
 <pinref part="R36" gate="G$1" pin="2"/>
 <wire x1="73.66" y1="73.66" x2="83.82" y2="73.66" width="0.1524" layer="91"/>
 </segment>
-<segment>
-<wire x1="78.74" y1="-30.48" x2="63.5" y2="-30.48" width="0.1524" layer="91"/>
-</segment>
 </net>
 <net name="CV2" class="0">
+<segment>
+<wire x1="78.74" y1="-33.02" x2="76.2" y2="-33.02" width="0.1524" layer="91"/>
+<pinref part="JP1" gate="A" pin="3"/>
+<wire x1="76.2" y1="-33.02" x2="63.5" y2="-33.02" width="0.1524" layer="91"/>
+<junction x="76.2" y="-33.02"/>
+</segment>
 <segment>
 <pinref part="R37" gate="G$1" pin="2"/>
 <wire x1="73.66" y1="50.8" x2="83.82" y2="50.8" width="0.1524" layer="91"/>
 </segment>
+</net>
+<net name="CV3" class="0">
 <segment>
-<wire x1="78.74" y1="-33.02" x2="63.5" y2="-33.02" width="0.1524" layer="91"/>
+<wire x1="78.74" y1="-35.56" x2="76.2" y2="-35.56" width="0.1524" layer="91"/>
+<pinref part="JP1" gate="A" pin="5"/>
+<wire x1="76.2" y1="-35.56" x2="63.5" y2="-35.56" width="0.1524" layer="91"/>
+<junction x="76.2" y="-35.56"/>
 </segment>
 </net>
-<net name="CV3" class="0">
+<net name="CV4" class="0">
+<segment>
+<wire x1="78.74" y1="-38.1" x2="76.2" y2="-38.1" width="0.1524" layer="91"/>
+<pinref part="JP1" gate="A" pin="7"/>
+<wire x1="76.2" y1="-38.1" x2="63.5" y2="-38.1" width="0.1524" layer="91"/>
+<junction x="76.2" y="-38.1"/>
+</segment>
 <segment>
 <pinref part="R38" gate="G$1" pin="2"/>
@@
 </segment>
 <segment>
-<wire x1="78.74" y1="-35.56" x2="63.5" y2="-35.56" width="0.1524" layer="91"/>
-</segment>
-</net>
-<net name="CV4" class="0">
-<segment>
 <pinref part="R39" gate="G$1" pin="2"/>
 <wire x1="73.66" y1="5.08" x2="83.82" y2="5.08" width="0.1524" layer="91"/>
 </segment>
-<segment>
-<wire x1="78.74" y1="-38.1" x2="63.5" y2="-38.1" width="0.1524" layer="91"/>
-</segment>
 </net>

Commit message: Schemas and layout updated
Parts:
- removed C20, C21, C26, C27, C30: 0.1uF, rcl:C-EUC0603
- removed C22, C23, C29: 10uF, rcl:CPOLRAD
- removed C24, C25: 1uF, rcl:CPOLRAD
- removed C28: (no value), rcl:C-USC1206
- removed CDCS502PW: CDCS502, components:CDCS502
- removed IC6: (no value), SparkFun-PowerIC:V_REG_TPS76433SOT23-5
- removed JP3: (no value), pinhead:PINHD-2X3
- removed PCM1808: PCM1808PW, Pekkas_libraries:PCM1808PW
- removed Q1: (no value), Pekkas_libraries:XTAL
- removed TLV71333: TVL713, Pekkas_libraries:TVL713
- added C33, C34, C35, C36, C37, C38, C39, C40: 0.1uF, resistor:C-EUC0603
Connections:
- removed net 3V3: C21.1, C23.+, C26.1, CDCS502PW.VDD, PCM1808.VDD, TLV71333.OUT
- removed net 5VCC: C20.1, C22.+, IC6.OUT, PCM1808.VCC
- removed net AGND: C20.2, C22.-
- removed net N$28: C25.+, PCM1808.VINL
- removed net N$29: CDCS502PW.XIN, Q1.1
- removed net N$3: C24.+, PCM1808.VINR
- removed net N$30: CDCS502PW.XOUT, Q1.2
- removed net N$31: C29.+, C30.1
- removed net N$32: CDCS502PW.CLK_OUT, PCM1808.SCK
- removed net N$33: JP3.1, PCM1808.LRCK
- removed net N$34: JP3.2, PCM1808.DOUT
- removed net N$35: JP3.3, PCM1808.BCK
- net +12VDC: now also C33.1, C34.1, C35.1, C36.1; no longer C28.1, IC6.EN, IC6.IN
- net -12VDC: now also C37.2, C38.2, C39.2, C40.2
- net 5VCON: no longer C27.1, TLV71333.EN, TLV71333.IN
- net CV1: now also R37.2; no longer R36.2
- net CV2: now also R36.2; no longer R37.2
- net CV3: now also R39.2
- net CV4: no longer R39.2
- net CV5: now also R42.2; no longer R40.2
- net CV6: now also R43.2; no longer R41.2
- net CV7: now also R40.2; no longer R42.2
- net CV8: now also R41.2; no longer R43.2
- net GND: now also C33.2, C34.2, C35.2, C36.2, C37.1, C38.1, C39.1, C40.1; no longer C21.2, C23.-, C26.2, C27.2, C28.2, C29.-, C30.2, CDCS502PW.FS, CDCS502PW.GND, CDCS502PW.SSC_SEL_0, CDCS502PW.SSC_SEL_1, IC6.GND, JP3.4, PCM1808.AGND, PCM1808.DGND, PCM1808.FMT, PCM1808.MD0, PCM1808.MD1, TLV71333.GND
Other:
- note removed: "Analog to digital conversion"
- note removed: "Caps for pcm1808"
- note removed: "Connector to RasPi"
- note removed: "PCM1808"
