File: Hardware/CV-Module CAD/CV-module-schematics.brd (EAGLE design)
At the start: 160 x 100 mm, 30 parts, among them U1 AD5611BKSZ, U2 AD5611BKSZ, U3 AD5611BKSZ, U4 AD5611BKSZ, U5 AD5611BKSZ, U6 AD5611BKSZ, U7 AD5611BKSZ, U8 AD5611BKSZ

Commit message: HW-design phase
Parts:
- removed U$2: POWER_SIMPLE10, eurorack:POWER_10
- added C17: 10uF, resistor:C1206
- added R10, R11, R4, R5, R6, R7, R8, R9: 20k, resistor:M1206
- added U$3: POWER, eurorack:POWER_16
Connections:
- new net N$3: C17.1, IC1.3, IC1.4, U$3.10, U$3.9
- new net VCC: C1.1, C10.1, C11.1, C12.1, C13.1, C15.1, C16.1, C2.1, C3.1, C4.1, C5.1, C6.1, C7.1, C8.1, C9.1, IC1.5, U1.4, U2.4, U3.4, U4.4, U5.4, U6.4, U7.4, U8.4
- net GND: now also C17.2, IC1.2, R11.2, R4.2, R5.2, R6.2, R7.2, R8.2, R9.2, U$1.6, U$1.7, U$1.8, U$3.3, U$3.4, U$3.5, U$3.6, U$3.7, U$3.8
- net SYNC1: now also R4.1
- net SYNC2: now also R5.1
- net SYNC3: now also R6.1
- net SYNC4: now also R7.1
- net SYNC5: now also R8.1
- net SYNC6: now also R9.1
- net SYNC7: now also R10.1
- net SYNC8: now also R11.1
- net VDD: now also U$1.16, U$1.3; no longer C1.1, C10.1, C11.1, C12.1, C13.1, C15.1, C16.1, C2.1, C3.1, C4.1, C5.1, C6.1, C7.1, C8.1, C9.1, IC1.5, U1.4, U2.4, U3.4, U4.4, U5.4, U6.4, U7.4, U8.4

Commit message: eagle project forward
Parts:
- added IC2, IC3, IC4, IC5: LM358D, linear:SO08
- added JP1: (no value), pinhead:2X04
- added R12, R13, R14, R15, R16, R17, R18, R19, R20, R21, R22, R23, R24, R25, R26, R27: 10k, resistor:R0603
- added R28, R29, R30, R31, R32, R33, R34, R35: (no value), pot:3223W
- added U9: (no value), SparkFun-PowerIC:SOT223
Connections:
- new net +5V: R28.2, U9.2, U9.4
- new net N$5: R12.1, R28.1
- new net V+: IC2.8, IC3.8, IC4.8, IC5.8
- new net V-: IC2.4, IC3.4, IC4.4, IC5.4
- net GND: now also U9.1
- net N$3: now also U9.3
Changed lines of the file:
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@@
 <element name="U$3" library="eurorack" package="POWER_16" value="POWER" x="-33.02" y="-193.04"/>
 <element name="C17" library="resistor" package="C1206" value="10uF" x="-39.37" y="-203.2"/>
+<element name="IC2" library="linear" package="SO08" value="LM358D" x="-46.99" y="-201.93"/>
+<element name="IC3" library="linear" package="SO08" value="LM358D" x="-55.88" y="-201.93"/>
+<element name="IC4" library="linear" package="SO08" value="LM358D" x="-64.77" y="-201.93"/>
+<element name="IC5" library="linear" package="SO08" value="LM358D" x="-73.66" y="-201.93"/>
+<element name="JP1" library="pinhead" package="2X04" value="" x="-72.39" y="-212.09"/>
+<element name="R12" library="resistor" package="R0603" value="10k" x="-76.2" y="-218.44"/>
+<element name="R13" library="resistor" package="R0603" value="10k" x="-76.2" y="-222.25"/>
+<element name="R14" library="resistor" package="R0603" value="10k" x="-76.2" y="-226.06"/>
+<element name="R15" library="resistor" package="R0603" value="10k" x="-76.2" y="-229.87"/>
+<element name="R16" library="resistor" package="R0603" value="10k" x="-76.2" y="-233.68"/>
+<element name="R17" library="resistor" package="R0603" value="10k" x="-76.2" y="-237.49"/>
+<element name="R18" library="resistor" package="R0603" value="10k" x="-76.2" y="-241.3"/>
+<element name="R19" library="resistor" package="R0603" value="10k" x="-76.2" y="-245.11"/>
+<element name="R20" library="resistor" package="R0603" value="10k" x="-76.2" y="-248.92"/>
+<element name="R21" library="resistor" package="R0603" value="10k" x="-76.2" y="-252.73"/>
+<element name="R22" library="resistor" package="R0603" value="10k" x="-76.2" y="-256.54"/>
+<element name="R23" library="resistor" package="R0603" value="10k" x="-76.2" y="-260.35"/>
+<element name="R24" library="resistor" package="R0603" value="10k" x="-76.2" y="-264.16"/>
+<element name="R25" library="resistor" package="R0603" value="10k" x="-76.2" y="-267.97"/>
+<element name="R26" library="resistor" package="R0603" value="10k" x="-76.2" y="-271.78"/>
+<element name="R27" library="resistor" package="R0603" value="10k" x="-76.2" y="-275.59"/>
+<element name="R28" library="pot" package="3223W" value="" x="-83.82" y="-273.05"/>
+<element name="R29" library="pot" package="3223W" value="" x="-91.44" y="-273.05"/>
+<element name="R30" library="pot" package="3223W" value="" x="-99.06" y="-273.05"/>
+<element name="R31" library="pot" package="3223W" value="" x="-106.68" y="-273.05"/>
+<element name="R32" library="pot" package="3223W" value="" x="-114.3" y="-273.05"/>
+<element name="R33" library="pot" package="3223W" value="" x="-121.92" y="-273.05"/>
+<element name="R34" library="pot" package="3223W" value="" x="-129.54" y="-273.05"/>
+<element name="R35" library="pot" package="3223W" value="" x="-137.16" y="-273.05"/>
+<element name="U9" library="SparkFun-PowerIC" package="SOT223" value="" x="-143.51" y="-273.05">
+<attribute name="PROD_ID" value="VREG-08170" x="-143.51" y="-273.05" size="1.778" layer="27" display="off"/>
+</element>
 </elements>
 <signals>
@@
 <contactref element="U$3" pad="7"/>
 <contactref element="C17" pad="2"/>
+<contactref element="U9" pad="1"/>
 <wire x1="-36.83" y1="-194.31" x2="-37.97" y2="-203.2" width="0" layer="19" extent="1-1"/>
 <wire x1="-36.83" y1="-191.77" x2="-36.83" y2="-194.31" width="0" layer="19" extent="1-1"/>
@@
 <wire x1="25.0444" y1="83.82" x2="27.5844" y2="73.66" width="0" layer="19" extent="1-1"/>
 <wire x1="60.6044" y1="52.07" x2="26.3144" y2="60.96" width="0" layer="19" extent="1-1"/>
+<wire x1="-145.8214" y1="-276.1488" x2="-37.97" y2="-203.2" width="0" layer="19" extent="1-1"/>
 </signal>
 <signal name="N$1">
@@
 <contactref element="IC1" pad="3"/>
 <contactref element="C17" pad="1"/>
+<contactref element="U9" pad="3"/>
 <wire x1="-29.21" y1="-194.31" x2="-40.77" y2="-203.2" width="0" layer="19" extent="1-1"/>
 <wire x1="-29.21" y1="-191.77" x2="-29.21" y2="-194.31" width="0" layer="19" extent="1-1"/>
+<wire x1="-141.1986" y1="-276.1488" x2="-40.77" y2="-203.2" width="0" layer="19" extent="1-1"/>
 <wire x1="-35.88" y1="-20.3501" x2="-29.21" y2="-191.77" width="0" layer="19" extent="1-1"/>
 <wire x1="-35.88" y1="-17.7499" x2="-35.88" y2="-20.3501" width="0" layer="19" extent="1-1"/>
@@
 <wire x1="60.6044" y1="51.4096" x2="26.3144" y2="60.2996" width="0" layer="19" extent="1-1"/>
 </signal>
+<signal name="V+">
+<contactref element="IC2" pad="8"/>
+<contactref element="IC3" pad="8"/>
+<contactref element="IC4" pad="8"/>
+<contactref element="IC5" pad="8"/>
+<wire x1="-57.785" y1="-199.33" x2="-48.895" y2="-199.33" width="0" layer="19" extent="1-1"/>
+<wire x1="-66.675" y1="-199.33" x2="-57.785" y2="-199.33" width="0" layer="19" extent="1-1"/>
+<wire x1="-75.565" y1="-199.33" x2="-66.675" y2="-199.33" width="0" layer="19" extent="1-1"/>
+</signal>
+<signal name="V-">
+<contactref element="IC2" pad="4"/>
+<contactref element="IC3" pad="4"/>
+<contactref element="IC4" pad="4"/>
+<contactref element="IC5" pad="4"/>
+<wire x1="-53.975" y1="-204.53" x2="-45.085" y2="-204.53" width="0" layer="19" extent="1-1"/>
+<wire x1="-62.865" y1="-204.53" x2="-53.975" y2="-204.53" width="0" layer="19" extent="1-1"/>
+<wire x1="-71.755" y1="-204.53" x2="-62.865" y2="-204.53" width="0" layer="19" extent="1-1"/>
+</signal>
+<signal name="+5V">
+<contactref element="U9" pad="2"/>
+<contactref element="U9" pad="4"/>
+<contactref element="R28" pad="2"/>
+<wire x1="-143.51" y1="-269.951" x2="-143.51" y2="-276.1488" width="0" layer="19" extent="1-1"/>
+<wire x1="-83.82" y1="-271.835" x2="-143.51" y2="-269.951" width="0" layer="19" extent="1-1"/>
+</signal>
+<signal name="N$5">
+<contactref element="R28" pad="1"/>
+<contactref element="R12" pad="1"/>
+<wire x1="-77.05" y1="-218.44" x2="-85.22" y2="-274.265" width="0" layer="19" extent="1-1"/>
+</signal>
 </signals>

Commit message: HW schematics and layout +parts updated
Parts:
- removed R10, R11, R9: 20k, resistor:M1206
- added C18, C19: 10uF, resistor:C1206
- added JP2: (no value), pinhead:2X03
- added R36, R37, R38, R39, R40, R41, R42, R43: 1k, resistor:R0603
- R1, R2, R3: value (none) -> 20k; device resistor:R1206 -> rcl:R0603
- R12, R14, R16, R18, R20, R22, R24, R26: value 10k -> 9.53k
- R4, R5, R6, R7, R8: device resistor:M1206 -> rcl:R0603
- moved R29 423.9 mm to (133.3, 86.4)
- moved R28 417.8 mm to (127.0, 87.6)
- moved R31 417.4 mm to (129.5, 71.1)
- moved R33 410.5 mm to (127.0, 53.3)
- moved R35 408.5 mm to (133.3, 33.0)
- moved R30 408.3 mm to (120.7, 71.1)
- moved R32 402.9 mm to (121.9, 53.3)
- moved R34 399.4 mm to (127.0, 33.0)
- moved R14 370.2 mm to (128.3, 82.5)
- moved R15 370.2 mm to (128.3, 78.7)
- moved R26 370.1 mm to (141.0, 27.9)
- moved R22 369.9 mm to (133.3, 48.3)
- moved R18 369.8 mm to (129.5, 66.0)
- moved R19 369.8 mm to (129.5, 62.2)
- moved R23 369.6 mm to (134.6, 43.2)
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Connections:
- removed net N$3: C17.1, IC1.3, IC1.4, U$3.10, U$3.9, U9.3
- removed net V+: IC2.8, IC3.8, IC4.8, IC5.8
- removed net V-: IC2.4, IC3.4, IC4.4, IC5.4
- new net +12VDC: C17.1, C19.1, IC1.3, IC1.4, IC2.8, IC3.8, IC4.8, IC5.8, U$3.10, U$3.9, U9.3
- new net -12VDC: IC2.4, IC3.4, IC4.4, IC5.4, U$3.1, U$3.2
- new net CTRL1: U$1.11
- new net CTRL2: U$1.10
- new net CTRL3: U$1.9
- new net CV1: R36.2
- new net CV2: R37.2
- new net CV3: R38.2
- new net CV4: R39.2
- new net CV5: JP1.2, R40.2
- new net CV6: JP1.4, R41.2
- new net CV7: JP1.6, R42.2
- new net CV8: JP1.8, R43.2
- new net N$10: R16.1, R30.1
- new net N$11: IC3.6, R18.2, R19.1
- new net N$12: R18.1, R31.1
- new net N$13: IC3.7, R19.2, R39.1
- new net N$14: IC3.1, R17.2, R38.1
- new net N$15: IC2.7, R15.2, R37.1
- new net N$16: IC4.2, R20.2, R21.1
- new net N$17: IC4.1, R21.2, R40.1
- new net N$18: IC4.7, R23.2, R41.1
- new net N$19: IC4.6, R22.2, R23.1
- new net N$20: IC5.2, R24.2, R25.1
- new net N$21: IC5.1, R25.2, R42.1
- new net N$22: R24.1, R34.1
- new net N$23: IC5.6, R26.2, R27.1
- new net N$24: IC5.7, R27.2, R43.1
- new net N$25: R26.1, R35.1
- new net N$26: R20.1, R32.1
- new net N$27: R22.1, R33.1
- new net N$4: IC2.2, R12.2, R13.1
- new net N$6: IC2.1, R13.2, R36.1
- new net N$7: R14.1, R29.1
- new net N$8: IC2.6, R14.2, R15.1
- new net N$9: IC3.2, R16.2, R17.1
- net +5V: now also C18.1, R29.2, R30.2, R31.2, R32.2, R33.2, R34.2, R35.2
- net GND: now also C18.2, C19.2, R1.2, R2.2, R3.2; no longer R11.2, R9.2
- net N$1: now also JP2.2, U1.3, U2.3, U3.3, U5.3, U6.3, U7.3, U8.3; no longer R2.2
- net N$2: now also JP2.4, U1.2, U2.2, U3.2, U5.2, U6.2, U7.2, U8.2; no longer R1.1
- net SYNC1: now also R1.1; no longer R4.1
- net SYNC2: now also R2.1; no longer R5.1
- net SYNC3: now also R3.1; no longer R6.1
- net SYNC4: now also R4.1; no longer R7.1
- net SYNC5: now also R5.1; no longer R8.1
- net SYNC6: now also R6.1; no longer R9.1
- net SYNC7: now also R7.1; no longer R10.1
- net SYNC8: now also R8.1; no longer R11.1
- net VDAC1: now also IC2.3
- net VDAC2: now also IC2.5
- net VDAC3: now also IC3.3
- net VDAC4: now also IC3.5
- net VDAC5: now also IC4.3
- net VDAC6: now also IC4.5
- net VDAC7: now also IC5.3
- net VDAC8: now also IC5.5

Commit message: Schema and Layout
Parts:
- added C20, C21: 0.1uF, rcl:C0603
- added C22, C23: 10uF, rcl:RADIALCAN4MM
- added C24, C25: 1uF, rcl:RADIALCAN4MM
- added U$2: PCM1808PW, Pekkas_libraries:R-PDSO-G14
- moved JP1 52.2 mm to (104.1, 47.0)
- moved IC2 48.9 mm to (68.6, 90.2)
- moved IC4 48.9 mm to (73.7, 52.1)
- moved R12 48.9 mm to (73.7, 91.4)
- moved R14 48.9 mm to (80.0, 90.2)
- moved R15 48.9 mm to (80.0, 86.4)
- moved R20 48.9 mm to (80.0, 55.9)
- moved R21 48.9 mm to (80.0, 50.8)
- moved R23 48.9 mm to (86.4, 50.8)
- moved R26 48.9 mm to (92.7, 35.6)
- moved R27 48.9 mm to (92.7, 30.5)
- moved R28 48.9 mm to (78.7, 95.2)
- moved R30 48.9 mm to (72.4, 78.7)
- moved R32 48.9 mm to (73.7, 61.0)
- moved R33 48.9 mm to (78.7, 61.0)
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
Commit message: layout forward
Parts:
- removed U$2: PCM1808PW, Pekkas_libraries:R-PDSO-G14
- added C26, C27, C30: 0.1uF, rcl:C0603
- added C28: (no value), rcl:C1206
- added C29: 10uF, rcl:RADIALCAN4MM
- added IC6: (no value), SparkFun-PowerIC:SOT23-5
- added JP3: (no value), pinhead:2X03
- added PCM1808: PCM1808PW, Pekkas_libraries:R-PDSO-G14
- added TLV71333: TVL713, Pekkas_libraries:SOT23-5
- moved C25 208.4 mm to (151.1, 90.2)
- moved C24 197.1 mm to (149.9, 82.5)
- moved C23 171.0 mm to (134.6, 69.8)
- moved C20 168.9 mm to (149.9, 64.8)
- moved C22 167.9 mm to (142.2, 62.2)
- moved C21 156.2 mm to (133.3, 66.0)
Connections:
- new net 3V3: C21.1, C23.1, C26.1, PCM1808.4, TLV71333.5
- new net 5VCC: C20.1, C22.1, IC6.5, PCM1808.3
- new net 5VCON: C27.1, TLV71333.1, TLV71333.3, U$3.11, U$3.12
- new net AGND: C20.2, C22.2
- new net N$28: C25.1, PCM1808.13
- new net N$3: C24.1, PCM1808.14
- new net N$31: C29.1, C30.1
- net +12VDC: now also C28.1, IC6.3, IC6.4
- net GND: now also C21.2, C23.2, C26.2, C27.2, C28.2, C29.2, C30.2, IC6.2, PCM1808.10, PCM1808.11, PCM1808.12, PCM1808.2, PCM1808.5, TLV71333.2

Commit message: Schema and layout design
Parts:
- added C31, C32: 10uF, resistor:C1206
- added CDCS502PW: CDCS502, components:SSOP-8
- added Q1: (no value), Pekkas_libraries:5X3CRYSTAL
- added U$2: TVL713, Pekkas_libraries:SOT23-5
- moved JP2 106.9 mm to (82.5, 7.62)
- moved JP1 103.4 mm to (10.2, 90.2)
- moved R1 85.9 mm to (85.1, 16.5), turned to 180 degrees
- moved JP3 82.5 mm to (142.2, 7.62)
- moved R2 80.7 mm to (85.1, 20.3), turned to 180 degrees
- moved R24 75.5 mm to (20.3, 69.8)
- moved R25 75.5 mm to (20.3, 66.0)
- moved R26 75.5 mm to (25.4, 69.8)
- moved R27 75.5 mm to (25.4, 64.8)
- moved R3 75.5 mm to (85.1, 24.1), turned to 180 degrees
- moved R42 75.5 mm to (31.8, 69.8)
- moved R43 75.5 mm to (30.5, 63.5)
- moved R4 70.4 mm to (85.1, 27.9), turned to 180 degrees
- moved R34 66.2 mm to (22.9, 76.2)
- moved R35 65.6 mm to (29.2, 74.9)
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Connections:
- removed net VDD: U$1.16, U$1.3
- new net 3V3MUX: C31.1, U$1.16, U$1.3, U$2.5
- new net N$29: CDCS502PW.1, Q1.1
- new net N$30: CDCS502PW.8, Q1.3
- new net N$32: CDCS502PW.6, PCM1808.6
- new net N$33: JP3.1, PCM1808.7
- new net N$34: JP3.2, PCM1808.9
- new net N$35: JP3.3, PCM1808.8
- net 3V3: now also CDCS502PW.7
- net 5VCON: now also C32.1, U$2.1, U$2.3
- net CTRL1: now also JP2.1
- net CTRL2: now also JP2.3
- net CTRL3: now also JP2.5
- net GND: now also C31.2, C32.2, CDCS502PW.2, CDCS502PW.3, CDCS502PW.4, CDCS502PW.5, JP3.4, U$2.2

Commit message: layout&schematics
Parts:
- moved R8 41.0 mm to (47.0, 27.9), turned to 90 degrees
- moved IC1 39.8 mm to (81.3, 21.6)
- moved R7 38.9 mm to (47.0, 31.8), turned to 270 degrees
- moved R6 37.7 mm to (49.3, 23.7), turned to 0 degrees
- moved U$3 35.6 mm to (96.5, 6.35)
- moved C17 35.1 mm to (81.3, 16.5), turned to 180 degrees
- moved R5 34.4 mm to (50.8, 34.3), turned to 90 degrees
- moved R4 31.8 mm to (54.6, 36.8), turned to 270 degrees
- moved R3 24.4 mm to (63.5, 35.5)
- moved U$2 24.3 mm to (71.1, 7.62), turned to 90 degrees
- moved R1 22.0 mm to (66.7, 28.5), turned to 90 degrees
- moved R2 21.7 mm to (67.2, 32.6), turned to 0 degrees
- moved JP2 20.9 mm to (62.2, 12.7), turned to 180 degrees
- moved C32 18.9 mm to (74.9, 6.35), turned to 90 degrees
- moved C1 14.0 mm to (76.2, 35.6), turned to 180 degrees
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Connections:
- net N$1: now also U4.3
- net N$2: now also U4.2
- net SYNC6: now also U8.1; no longer U6.1
- net SYNC7: now also U6.1; no longer U7.1
- net SYNC8: now also U7.1; no longer U8.1
- net VCC: now also C14.1
Routing:
- net GND: track 0.00 -> 165.8 mm, vias 0 -> 5
- net N$2: track 0.00 -> 163.0 mm, vias 0 -> 7
- net N$1: track 0.00 -> 139.3 mm, vias 0 -> 8
- net 3V3MUX: track 0.00 -> 42.0 mm
- net SYNC4: track 0.00 -> 41.4 mm, vias 0 -> 2
- net 5VCON: track 0.00 -> 35.5 mm
- net SYNC6: track 0.00 -> 25.0 mm
- net SYNC3: track 0.00 -> 18.9 mm
- net SYNC2: track 0.00 -> 14.9 mm
- net SYNC5: track 0.00 -> 14.9 mm
- net CTRL1: track 0.00 -> 14.7 mm
- net SYNC7: track 0.00 -> 14.2 mm
- net SYNC8: track 0.00 -> 14.1 mm
- net SYNC1: track 0.00 -> 12.5 mm
- net CTRL2: track 0.00 -> 11.6 mm
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
Commit message: HW
Parts:
- moved JP1 142.2 mm to (152.4, 88.9), turned to 90 degrees
- moved R32 128.4 mm to (147.3, 72.4), flipped to the bottom, turned to 270 degrees
- moved R21 128.3 mm to (152.4, 55.6), flipped to the bottom, turned to 270 degrees
- moved R20 128.2 mm to (152.3, 61.3), flipped to the bottom, turned to 270 degrees
- moved R40 120.7 mm to (155.8, 55.6), flipped to the bottom, turned to 90 degrees
- moved R24 119.3 mm to (138.9, 82.8), flipped to the bottom, turned to 270 degrees
- moved R25 119.0 mm to (138.8, 77.4), flipped to the bottom, turned to 270 degrees
- moved R33 117.6 mm to (141.0, 69.8), flipped to the bottom
- moved R23 113.5 mm to (145.3, 64.8), flipped to the bottom, turned to 90 degrees
- moved R34 112.9 mm to (134.2, 95.1), flipped to the bottom, turned to 270 degrees
- moved R22 112.7 mm to (142.4, 64.8), flipped to the bottom, turned to 270 degrees
- moved R42 110.8 mm to (142.3, 77.4), flipped to the bottom, turned to 90 degrees
- moved R41 110.0 mm to (148.2, 66.5), flipped to the bottom, turned to 90 degrees
- moved R27 108.5 mm to (131.7, 86.5), flipped to the bottom, turned to 90 degrees
- moved R43 106.9 mm to (134.4, 88.3), flipped to the bottom, turned to 90 degrees
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Connections:
- net CV1: now also JP1.1
- net CV2: now also JP1.3
- net CV3: now also JP1.5; no longer R38.2
- net CV4: now also JP1.7, R38.2
Routing:
- net VCC: track 0.00 -> 267.4 mm, vias 0 -> 2
- net GND: track 165.8 -> 407.4 mm, vias 5 -> 12
- net +5V: track 0.00 -> 26.1 mm
- net +12VDC: track 0.00 -> 19.3 mm
- net N$22: track 0.00 -> 15.4 mm
- net N$26: track 0.00 -> 13.9 mm
- net N$4: track 0.00 -> 12.8 mm
- net N$9: track 0.00 -> 11.9 mm
- net N$16: track 0.00 -> 11.6 mm
- net N$20: track 0.00 -> 11.0 mm
- net N$13: track 0.00 -> 10.3 mm
- net N$5: track 0.00 -> 9.84 mm
- net N$15: track 0.00 -> 9.62 mm
- net N$10: track 0.00 -> 9.47 mm
- net N$24: track 0.00 -> 9.00 mm
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