File: Hardware/CV-voltage conditioning/CV-module-schematics.sch (EAGLE design)
At the start: 62 parts, among them IC2 LM358D, IC3 LM358D, IC4 LM358D, IC5 LM358D

Commit message: updates
Parts:
- added JP3: (no value), pinhead:PINHD-1X3
Connections:
- net +12VDC: now also JP3.1
- net -12VDC: now also JP3.3
- net GND: now also JP3.2
Changed lines of the file:
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@@
 <part name="GND9" library="supply1" deviceset="GND" device=""/>
 <part name="GND10" library="supply1" deviceset="GND" device=""/>
+<part name="JP3" library="pinhead" deviceset="PINHD-1X3" device=""/>
 </parts>
 <sheets>
@@
 <instance part="GND9" gate="1" x="73.66" y="-50.8"/>
 <instance part="GND10" gate="1" x="55.88" y="91.44"/>
+<instance part="JP3" gate="A" x="-40.64" y="-43.18"/>
 </instances>
 <busses>
@@
 <junction x="12.7" y="-63.5"/>
 <label x="-1.016" y="-67.056" size="2.54" layer="95"/>
+<pinref part="JP3" gate="A" pin="3"/>
+<wire x1="-17.78" y1="-63.5" x2="-43.18" y2="-63.5" width="0.1524" layer="91"/>
+<wire x1="-43.18" y1="-63.5" x2="-43.18" y2="-45.72" width="0.1524" layer="91"/>
+<junction x="-17.78" y="-63.5"/>
 </segment>
 </net>
@@
 <junction x="-2.54" y="-22.86"/>
 <label x="-2.286" y="-22.352" size="2.54" layer="95"/>
+<wire x1="-17.78" y1="-22.86" x2="-35.56" y2="-22.86" width="0.1524" layer="91"/>
+<wire x1="-35.56" y1="-22.86" x2="-35.56" y2="-40.64" width="0.1524" layer="91"/>
+<junction x="-17.78" y="-22.86"/>
+<pinref part="JP3" gate="A" pin="1"/>
+<wire x1="-35.56" y1="-40.64" x2="-43.18" y2="-40.64" width="0.1524" layer="91"/>
 </segment>
 </net>
@@
 <wire x1="27.94" y1="-43.18" x2="45.72" y2="-43.18" width="0.1524" layer="91"/>
 <wire x1="45.72" y1="-43.18" x2="45.72" y2="-48.26" width="0.1524" layer="91"/>
-</segment>
-<segment>
+<wire x1="-17.78" y1="-43.18" x2="-43.18" y2="-43.18" width="0.1524" layer="91"/>
+<pinref part="JP3" gate="A" pin="2"/>
+</segment>
+<segment>

Commit message: updates for voltage-level module
Parts:
- added JP4: (no value), pinhead:PINHD-1X2
- added LM4120: LM4120, Pekkas_libraries:LM4120
- added R10: 39k, resistor:R-US_R0603
- added R9: 20k, resistor:R-US_R0603
Connections:
- new net N$34: JP4.1, LM4120.VOUT, R9.2
- net +12VDC: now also LM4120.EN, LM4120.VIN
- net +5V: now also JP4.2, R10.2, R9.1
- net GND: now also LM4120.GND, R10.1
Changed lines of the file:
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@@
 <part name="GND10" library="supply1" deviceset="GND" device=""/>
 <part name="JP3" library="pinhead" deviceset="PINHD-1X3" device=""/>
+<part name="LM4120" library="Pekkas_libraries" deviceset="LM4120" device=""/>
+<part name="GND11" library="supply1" deviceset="GND" device=""/>
+<part name="R9" library="resistor" deviceset="R-US_" device="R0603" value="20k"/>
+<part name="R10" library="resistor" deviceset="R-US_" device="R0603" value="39k"/>
+<part name="SUPPLY1" library="supply2" deviceset="+5V" device=""/>
+<part name="JP4" library="pinhead" deviceset="PINHD-1X2" device=""/>
 </parts>
 <sheets>
@@
 <plain>
 <text x="50.8" y="124.46" size="5.08" layer="91">Control-Voltage signal conditioning</text>
-<text x="119.38" y="-55.88" size="5.08" layer="91">CV outputs</text>
+<text x="76.2" y="-22.86" size="5.08" layer="91">CV outputs</text>
 </plain>
 <instances>
@@
 <instance part="GND10" gate="1" x="55.88" y="91.44"/>
 <instance part="JP3" gate="A" x="-40.64" y="-43.18"/>
+<instance part="LM4120" gate="G$1" x="-96.52" y="-2.54"/>
+<instance part="GND11" gate="1" x="-68.58" y="-33.02"/>
+<instance part="R9" gate="G$1" x="-68.58" y="-5.08" rot="R90"/>
+<instance part="R10" gate="G$1" x="-68.58" y="-20.32" rot="R90"/>
+<instance part="SUPPLY1" gate="+5V" x="-48.26" y="-2.54"/>
+<instance part="JP4" gate="G$1" x="-55.88" y="-5.08"/>
 </instances>
 <busses>
@@
 <pinref part="SUPPLY6" gate="+5V" pin="+5V"/>
 <wire x1="99.06" y1="68.58" x2="99.06" y2="71.12" width="0.1524" layer="91"/>
+</segment>
+<segment>
+<pinref part="R9" gate="G$1" pin="1"/>
+<pinref part="R10" gate="G$1" pin="2"/>
+<wire x1="-68.58" y1="-10.16" x2="-68.58" y2="-12.7" width="0.1524" layer="91"/>
+<wire x1="-68.58" y1="-12.7" x2="-68.58" y2="-15.24" width="0.1524" layer="91"/>
+<wire x1="-68.58" y1="-12.7" x2="-58.42" y2="-12.7" width="0.1524" layer="91"/>
+<junction x="-68.58" y="-12.7"/>
+<pinref part="SUPPLY1" gate="+5V" pin="+5V"/>
+<wire x1="-58.42" y1="-12.7" x2="-48.26" y2="-12.7" width="0.1524" layer="91"/>
+<wire x1="-48.26" y1="-12.7" x2="-48.26" y2="-5.08" width="0.1524" layer="91"/>
+<pinref part="JP4" gate="G$1" pin="2"/>
+<wire x1="-58.42" y1="-5.08" x2="-58.42" y2="-12.7" width="0.1524" layer="91"/>
+<junction x="-58.42" y="-12.7"/>
 </segment>
 </net>
@@
 <pinref part="JP3" gate="A" pin="1"/>
 <wire x1="-35.56" y1="-40.64" x2="-43.18" y2="-40.64" width="0.1524" layer="91"/>
+</segment>
+<segment>
+<pinref part="LM4120" gate="G$1" pin="VIN"/>
+<wire x1="-83.82" y1="-2.54" x2="-73.66" y2="-2.54" width="0.1524" layer="91"/>
+<label x="-82.296" y="-1.524" size="1.778" layer="95"/>
+<pinref part="LM4120" gate="G$1" pin="EN"/>
+<wire x1="-109.22" y1="-2.54" x2="-111.76" y2="-2.54" width="0.1524" layer="91"/>
+<wire x1="-111.76" y1="-2.54" x2="-111.76" y2="-7.62" width="0.1524" layer="91"/>
+<wire x1="-111.76" y1="-7.62" x2="-73.66" y2="-7.62" width="0.1524" layer="91"/>
+<wire x1="-73.66" y1="-7.62" x2="-73.66" y2="-2.54" width="0.1524" layer="91"/>
 </segment>
 </net>
@@
 <junction x="73.66" y="-45.72"/>
 </segment>
+<segment>
+<pinref part="R10" gate="G$1" pin="1"/>
+<pinref part="GND11" gate="1" pin="GND"/>
+<wire x1="-68.58" y1="-30.48" x2="-68.58" y2="-27.94" width="0.1524" layer="91"/>
+<pinref part="LM4120" gate="G$1" pin="GND"/>
+<wire x1="-68.58" y1="-27.94" x2="-68.58" y2="-25.4" width="0.1524" layer="91"/>
+<wire x1="-109.22" y1="0" x2="-114.3" y2="0" width="0.1524" layer="91"/>
+<wire x1="-114.3" y1="0" x2="-114.3" y2="-27.94" width="0.1524" layer="91"/>
+<wire x1="-114.3" y1="-27.94" x2="-68.58" y2="-27.94" width="0.1524" layer="91"/>
+<junction x="-68.58" y="-27.94"/>
+</segment>
 </net>
 <net name="CV3" class="0">
@@
 </segment>
 </net>
+<net name="N$34" class="0">
+<segment>
+<pinref part="LM4120" gate="G$1" pin="VOUT"/>
+<pinref part="R9" gate="G$1" pin="2"/>
+<wire x1="-83.82" y1="2.54" x2="-68.58" y2="2.54" width="0.1524" layer="91"/>
+<wire x1="-68.58" y1="2.54" x2="-68.58" y2="0" width="0.1524" layer="91"/>
+<pinref part="JP4" gate="G$1" pin="1"/>
+<wire x1="-58.42" y1="-2.54" x2="-58.42" y2="2.54" width="0.1524" layer="91"/>
+<wire x1="-58.42" y1="2.54" x2="-68.58" y2="2.54" width="0.1524" layer="91"/>
+<junction x="-68.58" y="2.54"/>
+</segment>
+</net>

Commit message: layouts
Parts:
- R28, R29, R30, R31, R32, R33, R34, R35: device pot:TRIM_EU-3223W -> Pekkas_libraries:TRIM_EU-3222W
Changed lines of the file:
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@@
 <part name="R26" library="resistor" deviceset="R-US_" device="R0603" value="9.53k"/>
 <part name="R27" library="resistor" deviceset="R-US_" device="R0603" value="10k"/>
-<part name="R28" library="pot" deviceset="TRIM_EU-" device="3223W"/>
-<part name="R29" library="pot" deviceset="TRIM_EU-" device="3223W"/>
-<part name="R30" library="pot" deviceset="TRIM_EU-" device="3223W"/>
-<part name="R31" library="pot" deviceset="TRIM_EU-" device="3223W"/>
-<part name="R32" library="pot" deviceset="TRIM_EU-" device="3223W"/>
-<part name="R33" library="pot" deviceset="TRIM_EU-" device="3223W"/>
-<part name="R34" library="pot" deviceset="TRIM_EU-" device="3223W"/>
-<part name="R35" library="pot" deviceset="TRIM_EU-" device="3223W"/>
+<part name="R28" library="Pekkas_libraries" deviceset="TRIM_EU-" device="3222W"/>
+<part name="R29" library="Pekkas_libraries" deviceset="TRIM_EU-" device="3222W"/>
+<part name="R30" library="Pekkas_libraries" deviceset="TRIM_EU-" device="3222W"/>
+<part name="R31" library="Pekkas_libraries" deviceset="TRIM_EU-" device="3222W"/>
+<part name="R32" library="Pekkas_libraries" deviceset="TRIM_EU-" device="3222W"/>
+<part name="R33" library="Pekkas_libraries" deviceset="TRIM_EU-" device="3222W"/>
+<part name="R34" library="Pekkas_libraries" deviceset="TRIM_EU-" device="3222W"/>
+<part name="R35" library="Pekkas_libraries" deviceset="TRIM_EU-" device="3222W"/>
 <part name="SUPPLY2" library="supply2" deviceset="+5V" device=""/>
 <part name="SUPPLY3" library="supply2" deviceset="+5V" device=""/>
