File: Hardware/ADC-Board/ADC-Board-schematics.brd (EAGLE design)
At the start: 61.9 x 47.7 mm, 44 parts, among them U2 OPA2348AIDCNTG4

Commit message: layout
Parts:
- moved C2 0.81 mm to (44.4, 23.4)
- moved C4 0.20 mm to (47.9, 29.3)
Routing:
- net GND: track 237.9 -> 244.1 mm
- net 5VCC: track 73.2 -> 72.0 mm
- net N$11: track 12.1 -> 13.2 mm
- net N$10: track 21.1 -> 22.0 mm
Other:
- board text added: "ADC-Board 1.0"
- board text removed: "AD-Converter"
